File: Hardware/CAN_Bridge.brd (EAGLE design)
At the start: 48.3 x 20.8 mm, 56 parts, among them IC1 REG1117, Q1 8 MHz, U1 STM32F405XXSTM32F405XX, U2 MCP2551-E/SN, U4 MCP2551-E/SN, X2 22-23-2021, X3 22-23-2031, X4 22-23-2031, X5 MINI-USB-32005-301

Commit message: new revision of hardware (minor changes)
Parts:
- removed C15, C21: 2u2, rcl:C0603
- removed C18: 100 n, rcl:C0603
- removed TP_RX, TP_TX: TPTP10SQ, testpad:TP10SQ
- moved R4 13.5 mm to (30.5, 8.32), turned to 180 degrees
- moved TP_SWCLK 5.33 mm to (14.0, 14.1)
- moved R13 4.13 mm to (14.0, 9.33), turned to 90 degrees
- moved R12 1.72 mm to (14.0, 12.3), turned to 270 degrees
- moved TP_SWDIO 1.71 mm to (15.6, 14.4)
- moved C16 1.31 mm to (29.0, 10.7), turned to 270 degrees
- moved C20 0.25 mm to (16.6, 0.38)
- moved R10 0.23 mm to (28.1, 0.76), turned to 180 degrees
- moved C19 0.20 mm to (28.1, 2.22)
- moved R19 0.18 mm to (30.0, 6.79)
- moved C22 0.13 mm to (15.9, -4.06)
- moved C23 0.13 mm to (30.5, 0.51)
- moved R11 0.06 mm to (17.5, 14.4)
- moved C17 0.06 mm to (29.7, 3.56)
Connections:
- removed net N$11: R4.2, U4.8
- removed net N$23: C21.1, U1.47
- removed net N$3: R2.2, U2.8
- removed net N$5: C15.1, U1.31
- removed net USART3_RX: TP_RX.TP, U1.30
- removed net USART3_TX: TP_TX.TP, U1.29
- net +3V3: now also R2.2, R4.2; no longer C18.1
- net CAN1_TX: now also R2.1
- net CAN2_TX: now also R4.1
- net GND: now also U1.31, U1.47, U2.8, U4.8; no longer C15.2, C18.2, C21.2, R2.1, R4.1
Routing:
- net +3V3: track 75.6 -> 87.5 mm
- net N$11: track 8.39 -> 0.00 mm
- net USART3_RX: track 5.15 -> 0.00 mm
- net N$23: track 4.25 -> 0.00 mm
- net N$3: track 3.69 -> 0.00 mm
- net N$5: track 2.91 -> 0.00 mm
- net USART3_TX: track 2.31 -> 0.00 mm
- net CAN2_TX: track 22.7 -> 23.7 mm
- net GND: track 40.9 -> 41.9 mm, vias 26 -> 25
- net CAN1_TX: track 14.4 -> 13.6 mm
