File: Hardware/CAN_Bridge.sch (EAGLE design)
At the start: 56 parts, among them IC1 REG1117, Q1 8 MHz, U1 STM32F405XXSTM32F405XX, U2 MCP2551-E/SN, U4 MCP2551-E/SN, X2 22-23-2021, X3 22-23-2031, X4 22-23-2031, X5 MINI-USB-32005-301

Commit message: new revision of hardware (minor changes)
Parts:
- removed C15, C21: 2u2, rcl:C-EUC0603
- removed C18: 100 n, rcl:C-EUC0603
- removed TP_RX, TP_TX: TPTP10SQ, testpad:TPTP10SQ
Connections:
- removed net N$11: R4.2, U4.RS
- removed net N$23: C21.1, U1.VCAP_2
- removed net N$3: R2.2, U2.RS
- removed net N$5: C15.1, U1.VCAP_1
- removed net USART3_RX: TP_RX.TP, U1.PB11
- removed net USART3_TX: TP_TX.TP, U1.PB10
- net +3V3: now also R2.2, R4.2; no longer C18.1
- net CAN1_TX: now also R2.1
- net CAN2_TX: now also R4.1
- net GND: now also U1.VCAP_1, U1.VCAP_2, U2.RS, U4.RS; no longer C15.2, C18.2, C21.2, R2.1, R4.1
Other:
- note removed: "0R for F0"
- moved on the sheet: R2, R4
